File: controller/pcb/terrarium.sch (KiCad schematic (older format))
At the start: 36 parts

Commit message: add v1.1 pcb
Parts:
- added R5: R_Small, Resistor_THT:R_Axial_DIN0207_L6.3mm_D2.5mm_P7.62mm_Horizontal, symbol Device:R_Small
- added TP1, TP2: TestPoint, symbol Connector:TestPoint
- R1, R2, R3, R4: footprint Resistor_THT:R_Axial_DIN0204_L3.6mm_D1.6mm_P2.54mm_Vertical -> Resistor_THT:R_Axial_DIN0207_L6.3mm_D2.5mm_P7.62mm_Horizontal
Connections:
- wire segments 105 -> 108
- no-connect marks 31 -> 32
Changed lines of the file:
@@
 F 0 "R1" V 6650 1950 50  0000 C CNN
 F 1 "R_Small" V 6450 1900 50  0000 C CNN
-F 2 "Resistor_THT:R_Axial_DIN0204_L3.6mm_D1.6mm_P2.54mm_Vertical" H 6550 1900 50  0001 C CNN
+F 2 "Resistor_THT:R_Axial_DIN0207_L6.3mm_D2.5mm_P7.62mm_Horizontal" H 6550 1900 50  0001 C CNN
 F 3 "~" H 6550 1900 50  0001 C CNN
 	1    6550 1900
@@
 F 0 "R3" V 6700 3550 50  0000 C CNN
 F 1 "R_Small" V 6500 3500 50  0000 C CNN
-F 2 "Resistor_THT:R_Axial_DIN0204_L3.6mm_D1.6mm_P2.54mm_Vertical" H 6600 3500 50  0001 C CNN
+F 2 "Resistor_THT:R_Axial_DIN0207_L6.3mm_D2.5mm_P7.62mm_Horizontal" H 6600 3500 50  0001 C CNN
 F 3 "~" H 6600 3500 50  0001 C CNN
 	1    6600 3500
@@
 F 0 "R4" V 7350 3650 50  0000 C CNN
 F 1 "R_Small" V 7150 3600 50  0000 C CNN
-F 2 "Resistor_THT:R_Axial_DIN0204_L3.6mm_D1.6mm_P2.54mm_Vertical" H 7250 3600 50  0001 C CNN
+F 2 "Resistor_THT:R_Axial_DIN0207_L6.3mm_D2.5mm_P7.62mm_Horizontal" H 7250 3600 50  0001 C CNN
 F 3 "~" H 7250 3600 50  0001 C CNN
 	1    7250 3600
@@
 F 0 "R2" V 7300 2050 50  0000 C CNN
 F 1 "R_Small" V 7100 2000 50  0000 C CNN
-F 2 "Resistor_THT:R_Axial_DIN0204_L3.6mm_D1.6mm_P2.54mm_Vertical" H 7200 2000 50  0001 C CNN
+F 2 "Resistor_THT:R_Axial_DIN0207_L6.3mm_D2.5mm_P7.62mm_Horizontal" H 7200 2000 50  0001 C CNN
 F 3 "~" H 7200 2000 50  0001 C CNN
 	1    7200 2000
@@
 	8150 2650 9000 2650
 $Comp
-L LED:WS2812B AD1
-U 1 1 6197A54B
-P 2850 6400
-F 0 "AD1" H 2900 6650 50  0000 L CNN
-F 1 "WS2812B" H 2850 6150 50  0000 L CNN
-F 2 "LED_SMD:LED_WS2812B_PLCC4_5.0x5.0mm_P3.2mm" H 2900 6100 50  0001 L TNN
-F 3 "https://cdn-shop.adafruit.com/datasheets/WS2812B.pdf" H 2950 6025 50  0001 L TNN
-	1    2850 6400
-	1    0    0    -1
-$EndComp
-$Comp
 L power:GND #PWR0136
 U 1 1 6197BC25
@@
 	1    0    0    -1
 $EndComp
-Wire Wire Line
-	2850 6700 2850 6800
 $Comp
 L power:+5V #PWR0137
@@
 Text GLabel 1200 4800 0    50   Input ~ 0
 G23
-Text GLabel 2400 6400 0    50   Input ~ 0
+Text GLabel 2400 6000 1    50   Input ~ 0
 G23
-Wire Wire Line
-	2400 6400 2550 6400
 $Comp
 L Device:C_Small C1
@@
 Wire Wire Line
 	3400 6800 2850 6800
+Wire Wire Line
+	2850 6800 2850 6850
+Wire Notes Line
+	3800 5750 3800 7100
+Wire Notes Line
+	700  5750 3800 5750
+Wire Notes Line
+	700  7100 3800 7100
+Wire Wire Line
+	2850 6700 2850 6800
 Connection ~ 2850 6800
-Wire Wire Line
-	2850 6800 2850 6850
-Wire Notes Line
-	3800 5750 3800 7100
-Wire Notes Line
-	700  5750 3800 5750
-Wire Notes Line
-	700  7100 3800 7100
+NoConn ~ 3150 6400
+$Comp
+L Device:R_Small R5
+U 1 1 61AECE35
+P 2400 6200
+F 0 "R5" V 2500 6200 50  0000 C CNN
+F 1 "R_Small" V 2300 6200 50  0000 C CNN
+F 2 "Resistor_THT:R_Axial_DIN0207_L6.3mm_D2.5mm_P7.62mm_Horizontal" H 2400 6200 50  0001 C CNN
+F 3 "~" H 2400 6200 50  0001 C CNN
+	1    2400 6200
+	1    0    0    -1
+$EndComp
+Wire Wire Line
+	2400 6100 2400 6050
+Wire Wire Line
+	2550 6400 2400 6400
+Wire Wire Line
+	2400 6400 2400 6300
+$Comp
+L Connector:TestPoint TP2
+U 1 1 61B1FAEF
+P 2400 6400
+F 0 "TP2" H 2450 6600 50  0000 R CNN
+F 1 "TestPoint" H 2342 6517 50  0001 R CNN
+F 2 "" H 2600 6400 50  0001 C CNN
+F 3 "~" H 2600 6400 50  0001 C CNN
+	1    2400 6400
+	-1   0    0    1
+$EndComp
+Connection ~ 2400 6400
+$Comp
+L Connector:TestPoint TP1
+U 1 1 61B2135A
+P 2400 6050
+F 0 "TP1" V 2400 6200 50  0000 L CNN
+F 1 "TestPoint" V 2450 6100 50  0001 L CNN
+F 2 "" H 2600 6050 50  0001 C CNN
+F 3 "~" H 2600 6050 50  0001 C CNN
+	1    2400 6050
+	0    1    1    0
+$EndComp
+Connection ~ 2400 6050
+Wire Wire Line
+	2400 6050 2400 6000
+$Comp
+L LED:WS2812B AD1
+U 1 1 6197A54B
+P 2850 6400
+F 0 "AD1" H 2900 6650 50  0000 L CNN
+F 1 "WS2812B" H 2850 6150 50  0000 L CNN
+F 2 "LED_SMD:LED_WS2812B_PLCC4_5.0x5.0mm_P3.2mm" H 2900 6100 50  0001 L TNN
+F 3 "https://cdn-shop.adafruit.com/datasheets/WS2812B.pdf" H 2950 6025 50  0001 L TNN
+	1    2850 6400
+	1    0    0    -1
+$EndComp
 $EndSCHEMATC

Commit message: add 3rd relay for lamp
Parts:
- removed S1, S2: Screw_Terminal_01x03, TerminalBlock:TerminalBlock_bornier-3_P5.08mm, symbol Connector:Screw_Terminal_01x03
- removed relay1: 1, Connector_PinHeader_2.54mm:PinHeader_1x03_P2.54mm_Vertical, symbol Connector_Generic_MountingPin:Conn_01x03_MountingPin
- removed relay2: 2, Connector_PinHeader_2.54mm:PinHeader_1x03_P2.54mm_Vertical, symbol Connector_Generic_MountingPin:Conn_01x03_MountingPin
- added D3: 1N47xxA, Diode_THT:D_DO-41_SOD81_P7.62mm_Horizontal, symbol Diode:1N47xxA
- added LED3: ACTIVE, LED_THT:LED_D3.0mm_Clear, symbol Device:LED
- added R6, R7: R_Small, Resistor_THT:R_Axial_DIN0207_L6.3mm_D2.5mm_P7.62mm_Horizontal, symbol Device:R_Small
- added RE3: SANYOU_SRD_Form_C, Relay_THT:Relay_SPDT_SANYOU_SRD_Series_Form_C, symbol Relay:SANYOU_SRD_Form_C
- added S0: Power 220 in, TerminalBlock:TerminalBlock_bornier-2_P5.08mm, symbol Connector:Screw_Terminal_01x02
- added S1: Heater 1 Out, TerminalBlock:TerminalBlock_bornier-2_P5.08mm, symbol Connector:Screw_Terminal_01x02
- added S2: Heater 2 Out, TerminalBlock:TerminalBlock_bornier-2_P5.08mm, symbol Connector:Screw_Terminal_01x02
- added S3: Lamp 1 Out, TerminalBlock:TerminalBlock_bornier-2_P5.08mm, symbol Connector:Screw_Terminal_01x02
- added TR3: MMBT3904, Package_TO_SOT_THT:TO-92, symbol Transistor_BJT:MMBT3904
- TP1, TP2: footprint (none) -> TestPoint:TestPoint_Pad_1.5x1.5mm
- renumbered AD1 to ALED1
Connections:
- net labels added: 220L, 220N, G14
- wire segments 108 -> 114
Other:
- note added: "Relays"
- note removed: "DIY Relays"
- note removed: "Daughter board relays"

Commit message: final changes in pcb v1.2
Parts:
- removed TP1, TP2: TestPoint, TestPoint:TestPoint_Pad_1.5x1.5mm, symbol Connector:TestPoint
- removed rxtx1: Conn_01x02, Connector_PinSocket_2.54mm:PinSocket_1x02_P2.54mm_Vertical, symbol Connector_Generic:Conn_01x02
- TR1, TR2, TR3: footprint Package_TO_SOT_THT:TO-92 -> Package_TO_SOT_THT:TO-92_Inline; symbol Transistor_BJT:MMBT3904 -> Transistor_BJT:S8050
Connections:
- wire segments 114 -> 120
Other:
- moved on the sheet: H1, H2, H3, H4, HT1, HT2, HT3, HT4, HT5, HT6

Commit message: fix labels
Parts:
- S1: value Heater 1 Out -> Lamp 1 Out
- S2: value Heater 2 Out -> Heater 1 Out
- S3: value Lamp 1 Out -> Heater 2 Out
Changed lines of the file:
@@
 P 9200 1250
 F 0 "S1" H 9280 1242 50  0000 L CNN
-F 1 "Heater 1 Out" H 9280 1151 50  0000 L CNN
+F 1 "Lamp 1 Out" H 9280 1151 50  0000 L CNN
 F 2 "TerminalBlock:TerminalBlock_bornier-2_P5.08mm" H 9200 1250 50  0001 C CNN
 F 3 "~" H 9200 1250 50  0001 C CNN
@@
 P 9200 2850
 F 0 "S2" H 9280 2842 50  0000 L CNN
-F 1 "Heater 2 Out" H 9280 2751 50  0000 L CNN
+F 1 "Heater 1 Out" H 9280 2751 50  0000 L CNN
 F 2 "TerminalBlock:TerminalBlock_bornier-2_P5.08mm" H 9200 2850 50  0001 C CNN
 F 3 "~" H 9200 2850 50  0001 C CNN
@@
 P 9200 4400
 F 0 "S3" H 9280 4392 50  0000 L CNN
-F 1 "Lamp 1 Out" H 9280 4301 50  0000 L CNN
+F 1 "Heater 2 Out" H 9280 4301 50  0000 L CNN
 F 2 "TerminalBlock:TerminalBlock_bornier-2_P5.08mm" H 9200 4400 50  0001 C CNN
 F 3 "~" H 9200 4400 50  0001 C CNN

Commit message: pcb v1.2 released
Parts:
- Q1: renamed from TR1; value MMBT3904 -> S8050
- Q2: renamed from TR2; value MMBT3904 -> S8050
- Q3: renamed from TR3; value MMBT3904 -> S8050
- R1, R3, R5, R7: value R_Small -> 150ohm
Connections:
- net G26: now reaches esp32-right1.10 (Pin_10)
- net G26: now also HT2.2 (Pin_2)
- net G25: now reaches esp32-right1.11 (Pin_11)
- net G25: now also LED1.2 (A)
- net G27: now reaches esp32-right1.9 (Pin_9)
- net G27: now also HT1.2 (Pin_2)
- net G14: no longer names the net of esp32-right1.8 (Pin_8)
- net G14: no longer LED1.2 (A)
- net G15: no longer names the net of esp32-left1.4 (Pin_4)
- net G15: no longer HT1.2 (Pin_2)
- net G2: no longer names the net of esp32-left1.5 (Pin_5)
- net G2: no longer HT2.2 (Pin_2)
Other:
- moved on the sheet: D1, D2, D3, H1, H2, H3, H4

Commit message: pcb: add rtc ds3231m
Parts:
- added BT1: LIR2032, Battery:BatteryHolder_Keystone_1058_1x2032, symbol Device:Battery_Cell
- added R8, R9: 4.7k, Resistor_THT:R_Axial_DIN0207_L6.3mm_D2.5mm_P7.62mm_Horizontal, symbol Device:R_Small
- added U1: DS3231M, Package_SO:SOIC-16W_7.5x10.3mm_P1.27mm, symbol Timer_RTC:DS3231M
Connections:
- net +3V3: now also R8.1, R9.2, U1.2 (VCC)
- net GND: now also BT1.2 (-), U1.10 (GND), U1.11 (GND), U1.12 (GND), U1.13 (GND), U1.5 (GND), U1.6 (GND), U1.7 (GND), U1.8 (GND), U1.9 (GND)
- net SCL: now also R9.1, U1.16 (SCL)
- net SDA: now also R8.2, U1.15 (SDA)
- new net: BT1.1 (+), U1.14 (VBAT)
- no-connect marks 32 -> 35
Changed lines of the file:
@@
 EELAYER 30 0
 EELAYER END
-$Descr A4 11693 8268
+$Descr A3 16535 11693
 encoding utf-8
 Sheet 1 1
@@
 Wire Wire Line
 	7350 1700 7350 1900
+$Comp
+L Timer_RTC:DS3231M U1
+U 1 1 61B87BF1
+P 2750 8450
+F 0 "U1" H 3100 8800 50  0000 C CNN
+F 1 "DS3231M" H 3000 8100 50  0000 C CNN
+F 2 "Package_SO:SOIC-16W_7.5x10.3mm_P1.27mm" H 2750 7850 50  0001 C CNN
+F 3 "http://datasheets.maximintegrated.com/en/ds/DS3231.pdf" H 3020 8500 50  0001 C CNN
+	1    2750 8450
+	1    0    0    -1
+$EndComp
+$Comp
+L power:GND #PWR0107
+U 1 1 61B962C0
+P 2750 9150
+F 0 "#PWR0107" H 2750 8900 50  0001 C CNN
+F 1 "GND" H 2755 8977 50  0000 C CNN
+F 2 "" H 2750 9150 50  0001 C CNN
+F 3 "" H 2750 9150 50  0001 C CNN
+	1    2750 9150
+	1    0    0    -1
+$EndComp
+Wire Wire Line
+	2750 8850 2750 9000
+$Comp
+L power:+3V3 #PWR0108
+U 1 1 61B9AE9E
+P 1600 7750
+F 0 "#PWR0108" H 1600 7600 50  0001 C CNN
+F 1 "+3V3" H 1615 7923 50  0000 C CNN
+F 2 "" H 1600 7750 50  0001 C CNN
+F 3 "" H 1600 7750 50  0001 C CNN
+	1    1600 7750
+	-1   0    0    -1
+$EndComp
+Wire Wire Line
+	2750 8050 2750 7750
+NoConn ~ 3250 8250
+NoConn ~ 3250 8550
+NoConn ~ 2250 8650
+Text GLabel 1650 8250 0    50   Input ~ 0
+SCL
+Text GLabel 1650 8350 0    50   Input ~ 0
+SDA
+Wire Wire Line
+	2650 7750 2650 8050
+$Comp
+L Device:Battery_Cell BT1
+U 1 1 61BCBE03
+P 3650 8450
+F 0 "BT1" H 3768 8546 50  0000 L CNN
+F 1 "LIR2032" H 3768 8455 50  0000 L CNN
+F 2 "Battery:BatteryHolder_Keystone_1058_1x2032" V 3650 8510 50  0001 C CNN
+F 3 "~" V 3650 8510 50  0001 C CNN
+	1    3650 8450
+	1    0    0    -1
+$EndComp
+Wire Wire Line
+	3650 8250 3650 7750
+Wire Wire Line
+	2750 7750 3650 7750
+Wire Wire Line
+	3650 8550 3650 9000
+Wire Wire Line
+	3650 9000 2750 9000
+Connection ~ 2750 9000
+Wire Wire Line
+	2750 9000 2750 9150
+$Comp
+L Device:R_Small R9
+U 1 1 61BDE005
+P 2050 7950
+F 0 "R9" H 2150 7950 50  0000 C CNN
+F 1 "4.7k" V 1950 7950 50  0000 C CNN
+F 2 "Resistor_THT:R_Axial_DIN0207_L6.3mm_D2.5mm_P7.62mm_Horizontal" H 2050 7950 50  0001 C CNN
+F 3 "~" H 2050 7950 50  0001 C CNN
+	1    2050 7950
+	-1   0    0    1
+$EndComp
+$Comp
+L Device:R_Small R8
+U 1 1 61BDEC6F
+P 2000 8500
+F 0 "R8" V 2100 8500 50  0000 C CNN
+F 1 "4.7k" V 1900 8500 50  0000 C CNN
+F 2 "Resistor_THT:R_Axial_DIN0207_L6.3mm_D2.5mm_P7.62mm_Horizontal" H 2000 8500 50  0001 C CNN
+F 3 "~" H 2000 8500 50  0001 C CNN
+	1    2000 8500
+	0    -1   -1   0
+$EndComp
+Wire Wire Line
+	2250 8350 2200 8350
+Wire Wire Line
+	2250 8250 2050 8250
+Wire Wire Line
+	2050 7750 2050 7850
+Connection ~ 2050 7750
+Wire Wire Line
+	2050 7750 2650 7750
+Wire Wire Line
+	2050 8050 2050 8250
+Connection ~ 2050 8250
+Wire Wire Line
+	2050 8250 1650 8250
+Wire Wire Line
+	1600 7750 1800 7750
+Wire Wire Line
+	1900 8500 1800 8500
+Wire Wire Line
+	1800 8500 1800 7750
+Connection ~ 1800 7750
+Wire Wire Line
+	1800 7750 2050 7750
+Wire Wire Line
+	2100 8500 2200 8500
+Wire Wire Line
+	2200 8500 2200 8350
+Connection ~ 2200 8350
+Wire Wire Line
+	2200 8350 1650 8350
 $EndSCHEMATC

Commit message: pcb: add esp32
Parts:
- removed esp32-left1, esp32-right1: Conn_01x19_MountingPin, Connector_PinHeader_2.54mm:PinHeader_1x19_P2.54mm_Vertical, symbol Connector_Generic_MountingPin:Conn_01x19_MountingPin
- removed i2c1: RTC, Connector_PinHeader_2.54mm:PinHeader_1x04_P2.54mm_Vertical, symbol Connector_Generic:Conn_01x04
- added C2: 10uF, Capacitor_THT:C_Disc_D5.0mm_W2.5mm_P5.00mm, symbol Device:C_Small
- added C3: 47uF, Capacitor_THT:C_Disc_D5.0mm_W2.5mm_P5.00mm, symbol Device:C_Small
- added CONN1: data, Connector_PinHeader_2.54mm:PinHeader_1x04_P2.54mm_Vertical, symbol Connector_Generic:Conn_01x04
- added LED4: POWER, LED_THT:LED_D3.0mm_Clear, symbol Device:LED
- added R10, R11: 10k, Resistor_THT:R_Axial_DIN0207_L6.3mm_D2.5mm_P7.62mm_Horizontal, symbol Device:R_Small
- added R12: 300, Resistor_THT:R_Axial_DIN0207_L6.3mm_D2.5mm_P7.62mm_Horizontal, symbol Device:R_Small
- added S4: 5v in, TerminalBlock:TerminalBlock_bornier-2_P5.08mm, symbol Connector:Screw_Terminal_01x02
- added SW1, SW2: SW_Push, Button_Switch_SMD:SW_DIP_SPSTx01_Slide_6.7x4.1mm_W6.73mm_P2.54mm_LowProfile_JPin, symbol Switch:SW_Push
- added U1: ESP32-WROOM-32, RF_Module:ESP32-WROOM-32, symbol RF_Module:ESP32-WROOM-32
- added U3: LM1117-3.3, Package_TO_SOT_SMD:SOT-223-3_TabPin2, symbol Regulator_Linear:LM1117-3.3
- renumbered U1 to U2
Connections:
- net +3V3: now also C3.1, CONN1.1 (Pin_1), LED4.2 (A), R10.1, R11.1, U1.2 (VDD), U3.2 (VO)
- net +5V: now also C2.1, S4.2 (Pin_2), U3.3 (VI)
- net G16: now also HT6.2 (Pin_2), U1.27 (IO16); no longer HT3.2 (Pin_2)
- net G17: now also HT5.2 (Pin_2), U1.28 (IO17); no longer HT4.2 (Pin_2)
- net G18: now also HT4.2 (Pin_2), U1.30 (IO18); no longer HT5.2 (Pin_2)
- net G19: now also HT3.2 (Pin_2), U1.31 (IO19); no longer HT6.2 (Pin_2)
- net G23: now also U1.37 (IO23)
- net G25: now also LED3.2 (A), U1.10 (IO25); no longer LED1.2 (A)
- net G26: now also HT1.2 (Pin_2), U1.11 (IO26); no longer HT2.2 (Pin_2)
- net G27: now also HT2.2 (Pin_2), U1.12 (IO27); no longer HT1.2 (Pin_2)
- net G4: now also U1.26 (IO4)
- net G5: now also LED1.2 (A), U1.29 (IO5); no longer LED3.2 (A)
- net GND: now also C2.2, C3.2, CONN1.4 (Pin_4), R12.1, S4.1 (Pin_1), SW1.1, SW2.2, U1.1 (GND), U1.15 (GND), U1.38 (GND), U1.39 (GND), U3.1 (GND)
- net RX: now also CONN1.3 (Pin_3), U1.34 (RXD0/IO3)
- net SCL: now also U1.36 (IO22)
- net SDA: now also U1.33 (IO21)
- net TX: now also CONN1.2 (Pin_2), U1.35 (TXD0/IO1)
- new net: R10.2, SW2.1, U1.25 (IO0)
- new net: R11.2, SW1.2, U1.3 (EN)
- new net: LED4.1 (K), R12.2
- no-connect marks 35 -> 30
Other:
- note removed: "esp32"
- moved on the sheet: BT1, R8, R9, U2
