File: controller/pcb/usb_and_cp2102.sch (KiCad schematic (older format))
At the start: 13 parts, among them P1 USB_C_Plug_USB2.0, Q5 BC817, Q6 BC817, U3 LM1117-3.3, U4 CP2102N-A02-GQFN28

Commit message: move components around
Parts:
- added C10: 0.47uF, Capacitor_SMD:C_1206_3216Metric, symbol Device:C_Small
- Q5, Q6: value BC817 -> s8050
- R19, R20: value 10k -> 150
Connections:
- net EN: now also C10.1
- net GND: now also C10.2
Changed lines of the file:
@@
 P 4050 5550
 F 0 "Q6" H 4241 5504 50  0000 L CNN
-F 1 "BC817" H 4241 5595 50  0000 L CNN
+F 1 "s8050" H 4241 5595 50  0000 L CNN
 F 2 "Package_TO_SOT_SMD:SOT-23" H 4250 5475 50  0001 L CIN
 F 3 "https://www.onsemi.com/pub/Collateral/BC818-D.pdf" H 4050 5550 50  0001 L CNN
@@
 AR Path="/623D759E/6245B6BE" Ref="R20"  Part="1"
 F 0 "R20" V 3850 5550 50  0000 C CNN
-F 1 "10k" V 3650 5550 50  0000 C CNN
+F 1 "150" V 3650 5550 50  0000 C CNN
 F 2 "Resistor_SMD:R_1206_3216Metric" H 3750 5550 50  0001 C CNN
 F 3 "~" H 3750 5550 50  0001 C CNN
@@
 AR Path="/623D759E/6245AA5F" Ref="R19"  Part="1"
 F 0 "R19" V 3850 6150 50  0000 C CNN
-F 1 "10k" V 3650 6150 50  0000 C CNN
+F 1 "150" V 3650 6150 50  0000 C CNN
 F 2 "Resistor_SMD:R_1206_3216Metric" H 3750 6150 50  0001 C CNN
 F 3 "~" H 3750 6150 50  0001 C CNN
@@
 P 4050 6150
 F 0 "Q5" H 4241 6196 50  0000 L CNN
-F 1 "BC817" H 4241 6105 50  0000 L CNN
+F 1 "s8050" H 4241 6105 50  0000 L CNN
 F 2 "Package_TO_SOT_SMD:SOT-23" H 4250 6075 50  0001 L CIN
 F 3 "https://www.onsemi.com/pub/Collateral/BC818-D.pdf" H 4050 6150 50  0001 L CNN
@@
 Wire Wire Line
 	2400 4500 2200 4500
+$Comp
+L Device:C_Small C?
+U 1 1 623F3F18
+P 4150 6600
+AR Path="/623F3F18" Ref="C?"  Part="1"
+AR Path="/623D759E/623F3F18" Ref="C10"  Part="1"
+F 0 "C10" H 4242 6646 50  0000 L CNN
+F 1 "0.47uF" H 4242 6555 50  0000 L CNN
+F 2 "Capacitor_SMD:C_1206_3216Metric" H 4150 6600 50  0001 C CNN
+F 3 "~" H 4150 6600 50  0001 C CNN
+	1    4150 6600
+	1    0    0    -1
+$EndComp
+$Comp
+L power:GND #PWR?
+U 1 1 623F58EB
+P 4150 6850
+AR Path="/623F58EB" Ref="#PWR?"  Part="1"
+AR Path="/623D759E/623F58EB" Ref="#PWR019"  Part="1"
+F 0 "#PWR019" H 4150 6600 50  0001 C CNN
+F 1 "GND" H 4155 6677 50  0000 C CNN
+F 2 "" H 4150 6850 50  0001 C CNN
+F 3 "" H 4150 6850 50  0001 C CNN
+	1    4150 6850
+	1    0    0    -1
+$EndComp
+Wire Wire Line
+	4150 6850 4150 6700
+Wire Wire Line
+	4150 6500 4150 6400
+Connection ~ 4150 6400
 $EndSCHEMATC
